Commit message: fix: restore simulated IMU publishing

File: src/amr_simulation/models/turtlebot3_waffle_rgbd.sdf.xacro (robot description, xacro)
@@ -406,4 +406,9 @@
         <pose>0.0 0.0 0.010 0 0 0</pose>
       </joint>
+      <joint name="imu_joint" type="fixed">
+        <parent>base_link</parent>
+        <child>imu_link</child>
+        <pose>0.0 0.0 0.068 0 0 0</pose>
+      </joint>
       <joint name="wheel_left_joint" type="revolute">
         <parent>base_link</parent>
